Commit message: feat: urdf for sm3

File: urdf/laboratory/sm3_laser.urdf (robot description, URDF)
Before this commit: robot bluerov2_heavy, 3 links, 2 joints
Links:
- link base_link: geometry 
Joints:
- joint left_camera_joint: origin xyz=0.048 0.153 0 rpy=-1.5707 0.1760 -1.5707 -> xyz=0 0.153 0.0 rpy=-1.5707 0 -1.7467
- joint right_camera_joint: origin xyz=0.0 -0.153 0 rpy=-1.5707 -0.1760 -1.5707 -> xyz=0.0 -0.153 0 rpy=-1.5707 0 -1.3947
