Commit message: refactor: update git

File: urdf/laboratory/optical_test_bench.urdf (robot description, URDF)
Before this commit: robot optical_bench, 7 links, 6 joints
Links:
- removed link SM3/base_link
- removed link SM3/left_camera_link
- removed link SM3/right_camera_link
- added link Passive/base_link; visual box size=0.035 0.220 0.005
- added link Passive/left_camera_link; visual cylinder length=0.05 radius=0.01
- added link Passive/right_camera_link; visual cylinder length=0.05 radius=0.01
- added link SM4/laser_link; visual box size=0.045 0.045 0.07
- added link SM4/projector_link; visual box size=0.15 0.15 0.03
- added link left_base_link; visual box size=0.045 0.245 0.045
- added link right_base_link; visual box size=0.045 0.245 0.045
- link SM4/base_link: geometry visual box size=0.045 0.52 0.045
Joints:
- removed joint SM3/base_joint
- removed joint SM3/left_camera_joint
- removed joint SM3/right_camera_joint
- removed joint SM4/base_joint
- added joint Passive/base_joint: type fixed, parent base_link, child Passive/base_link, origin xyz=0 0 0.295 rpy=0 0 0
- added joint Passive/left_camera_joint: type fixed, parent Passive/base_link, child Passive/left_camera_link, origin xyz=0 0.1 0.0125 rpy=-1.5707 0 -1.5707
- added joint Passive/right_camera_joint: type fixed, parent Passive/base_link, child Passive/right_camera_link, origin xyz=0.0 -0.1 0.0125 rpy=-1.5707 0 -1.5707
- added joint SM4/laser_joint: type fixed, parent SM4/base_link, child SM4/laser_link, origin xyz=0.0 0.0 0.0675 rpy=-1.5707 0 -1.5707
- added joint SM4/projector_joint: type fixed, parent SM4/base_link, child SM4/projector_link, origin xyz=0.0 0.0 -0.0475 rpy=-1.5 0 -1.5707
- added joint base_joint: type fixed, parent base_link, child SM4/base_link, origin xyz=-0 0 0.2 rpy=0 0 0
- added joint left_base_joint: type fixed, parent SM4/base_link, child left_base_link, origin xyz=0 0.2825 -0.0775 rpy=0 0 0
- added joint right_base_joint: type fixed, parent SM4/base_link, child right_base_link, origin xyz=0 -0.2825 -0.0775 rpy=0 0 0
- joint SM4/left_camera_joint: origin xyz=0 0.1627 0.0 rpy=-1.5707 0 -1.7129 -> xyz=0 0.15 0.0325 rpy=-1.5707 0 -1.5707
- joint SM4/right_camera_joint: origin xyz=0.0 -0.1627 0 rpy=-1.5707 0 -1.4285 -> xyz=0.0 -0.15 0.0325 rpy=-1.5707 0 -1.5707
