Commit message: feat: add base_link equal to camera frame

File: urdf/laboratory/mobile_bench.urdf (robot description, URDF)
Before this commit: robot mobile_bench, 11 links, 10 joints
Links:
- added link base_link_cam
- added link base_link_ned
Joints:
- added joint base_cam_joint: type fixed, parent base_link, child base_link_cam, origin xyz=0 0 0 rpy=-1.5707 0 -1.5707
- added joint base_ned_joint: type fixed, parent base_link, child base_link_ned, origin xyz=0 0 0 rpy=3.14

File: urdf/laboratory/optical_test_bench.urdf (robot description, URDF)
Before this commit: robot optical_bench, 11 links, 10 joints
Links:
- added link base_link_cam
Joints:
- added joint base_ned_joint: type fixed, parent base_link, child base_link_cam, origin xyz=0 0 0 rpy=-1.5707 0 -1.5707

Commit message: feat: improve mobile_bench.urdf to represent the CAD

File: urdf/laboratory/mobile_bench.urdf (robot description, URDF)
Before this commit: robot mobile_bench, 13 links, 12 joints
Links:
- removed link Active/SM3/laser_link
- removed link Active/SM4/projector_link
- removed link base_left_link
- removed link base_right_link
- added link navigation_link
- link Active/base_link: geometry 
- link Passive/base_link: geometry 
- link base_link: geometry visual mesh filename=package://voris_description/urdf/meshes/lab_bench.dae scale=1 1 1
Joints:
- removed joint Active/SM3/laser_joint
- removed joint Active/SM4/projector_joint
- removed joint base_left_joint
- removed joint base_right_joint
- removed joint left_base_joint
- added joint Active/base_link_joint: type fixed, parent base_link, child Active/base_link, origin xyz=-0 0 0.297 rpy=0 0 0
- added joint base_nav_joint: type fixed, parent base_link, child navigation_link, origin xyz=0.08 0 0.064 rpy=0 0 0
- joint Active/left_camera_joint: origin xyz=0 0.1863 0.0325 rpy=-1.5707 0 -1.7557 -> xyz=0 0.1863 0.0 rpy=-1.5707 0 -1.7557
- joint Active/right_camera_joint: origin xyz=0.0 -0.1863 0.0325 rpy=-1.5707 0 -1.3857 -> xyz=0.0 -0.1863 0.0 rpy=-1.5707 0 -1.3857
- joint Passive/base_joint: origin xyz=0 0 0.387 rpy=0 0 0 -> xyz=0 0 0.064 rpy=0 0 0; parent base_link -> Active/base_link
- joint Passive/left_camera_joint: origin xyz=0 0.1 0.0125 rpy=-1.5707 0 -1.5707 -> xyz=0 0.1 0 rpy=-1.5707 0 -1.5707
- joint Passive/right_camera_joint: origin xyz=0.0 -0.1 0.0125 rpy=-1.5707 0 -1.5707 -> xyz=0.0 -0.1 0 rpy=-1.5707 0 -1.5707

Commit message: feat: update transform between passive and active system

File: urdf/laboratory/mobile_bench.urdf (robot description, URDF)
Before this commit: robot mobile_bench, 10 links, 9 joints
Joints:
- joint Active/base_link_joint: origin xyz=-0 0 0.297 rpy=0 0 0 -> xyz=0 0 0.297 rpy=0 0 0
- joint Active/left_camera_joint: origin xyz=0 0.1863 0.0 rpy=-1.5707 0 -1.7557 -> xyz=0 0.2 0.0 rpy=-1.5707 0 -1.8722
- joint Active/right_camera_joint: origin xyz=0.0 -0.1863 0.0 rpy=-1.5707 0 -1.3857 -> xyz=0.0 -0.2 0.0 rpy=-1.5707 0 -1.1926
- joint Passive/base_joint: origin xyz=0 0 0.064 rpy=0 0 0 -> xyz=0.08 0 0.064 rpy=0 0 0

Commit message: refactor mobile bench urdf and cmakelist to remove include folder

File: urdf/laboratory/mobile_bench.urdf (robot description, URDF)
Before this commit: robot mobile_bench, 10 links, 9 joints
Joints:
- joint Passive/base_joint: origin xyz=0.08 0 0.064 rpy=0 0 0 -> xyz=0.008 0 0.064 rpy=0 0 0
