Commit message: feat: publishing joint_state from gazebo

File: urdf/bluerov2/simple_bluerov2_heavy.urdf (robot description, URDF)
Before this commit: robot bluerov2_heavy, 3 links, 2 joints
Links:
- added link thruster1_link; visual cylinder length=0.02 radius=0.05
- link base_link: geometry visual box size=0.05 0.05 0.1
Joints:
- added joint thruster1_joint: type continuous, parent base_link, child thruster1_link, origin xyz=0.138 -0.098 -0.0137 rpy=-1.570 1.570 -0.785, axis 0 0 1

Commit message: feat: publishing robot_description with all propellers or not based on launch arguments

File: urdf/bluerov2/simple_bluerov2_heavy.urdf (robot description, URDF)
Before this commit: robot bluerov2_heavy, 4 links, 3 joints
Links:
- removed link thruster1_link
- link base_link: geometry visual mesh filename=package://voris_description/urdf/meshes/bluerov2_heavy_skid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 scale=1 1 1
- link left_camera_link: geometry visual cylinder length=0.02 radius=0.01
- link right_camera_link: geometry visual cylinder length=0.02 radius=0.01
Joints:
- removed joint thruster1_joint
- joint left_camera_joint: origin xyz=0.19 0.075 0.201 rpy=-1.57 0 -1.57 -> xyz=0.19 0.075 0.201 rpy=-1.5707 0 -1.5707
- joint right_camera_joint: origin xyz=0.19 -0.075 0.201 rpy=-1.57 0 -1.57 -> xyz=0.19 -0.075 0.201 rpy=-1.5707 0 -1.5707

Commit message: feat: add cameras rotated frames

File: urdf/bluerov2/simple_bluerov2_heavy.urdf (robot description, URDF)
Before this commit: robot bluerov2_heavy, 3 links, 2 joints
Links:
- added link left_camera_frame
- added link right_camera_frame
Joints:
- added joint left_link_to_frame_joint: type fixed, parent left_camera_link, child left_camera_frame, origin xyz=0 0 0 rpy=-1.5707 0 -1.5707
- added joint right_link_to_frame_joint: type fixed, parent right_camera_link, child right_camera_frame, origin xyz=0 0 0 rpy=-1.5707 0 -1.5707
- joint left_camera_joint: origin xyz=0.19 0.075 0.201 rpy=-1.5707 0 -1.5707 -> xyz=0.19 0.075 0.201 rpy=0 0 0
- joint right_camera_joint: origin xyz=0.19 -0.075 0.201 rpy=-1.5707 0 -1.5707 -> xyz=0.19 -0.075 0.201 rpy=0 0 0

Commit message: feat: update cameras link position based on first extrinsic calibration

File: urdf/bluerov2/simple_bluerov2_heavy.urdf (robot description, URDF)
Before this commit: robot bluerov2_heavy, 5 links, 4 joints
Links:
- removed link left_camera_frame
- removed link left_camera_link
- removed link right_camera_frame
- removed link right_camera_link
- added link Passive/left_camera_link
- added link Passive/right_camera_link
Joints:
- removed joint left_link_to_frame_joint
- removed joint right_link_to_frame_joint
- joint left_camera_joint: child left_camera_link -> Passive/left_camera_link; origin xyz=0.19 0.075 0.201 rpy=0 0 0 -> xyz=0.19 0.075 0.201 rpy=-1.5707 0 -1.5707
- joint right_camera_joint: child right_camera_link -> Passive/right_camera_link; origin xyz=0.19 -0.075 0.201 rpy=0 0 0 -> xyz=0.19 -0.075 0.201 rpy=-1.5707 0 -1.5707

File: urdf/laboratory/mobile_bench.urdf (robot description, URDF)
Before this commit: robot mobile_bench, 13 links, 12 joints
Links:
- link base_left_link: geometry visual box size=0.045 0.34 0.045
- link base_right_link: geometry visual box size=0.045 0.34 0.045
Joints:
- joint Active/left_camera_joint: origin xyz=0 0.15 0.0325 rpy=-1.5707 0 -1.5707 -> xyz=0 0.1863 0.0325 rpy=-1.5707 0 -1.7557
- joint Active/right_camera_joint: origin xyz=0.0 -0.15 0.0325 rpy=-1.5707 0 -1.5707 -> xyz=0.0 -0.1863 0.0325 rpy=-1.5707 0 -1.3857
- joint Passive/base_joint: origin xyz=0 0 0.295 rpy=0 0 0 -> xyz=0 0 0.387 rpy=0 0 0
- joint base_left_joint: origin xyz=0 0.2825 -0.0775 rpy=0 0 0 -> xyz=0 0.2825 -0.14 rpy=0 0 0
- joint base_ned_joint: origin xyz=0 0 0 rpy=3.14 -> xyz=0 0 0 rpy=3.14 0 0
- joint base_right_joint: origin xyz=0 -0.2825 -0.0775 rpy=0 0 0 -> xyz=0 -0.2825 -0.14 rpy=0 0 0
- joint left_base_joint: origin xyz=-0 0 0.2 rpy=0 0 0 -> xyz=-0 0 0.305 rpy=0 0 0

Commit message: feat: add enu camera frames

File: urdf/bluerov2/simple_bluerov2_heavy.urdf (robot description, URDF)
Before this commit: robot bluerov2_heavy, 3 links, 2 joints
Links:
- added link Passive/left_camera_enu_link
- added link Passive/right_camera_enu_link
Joints:
- added joint left_camera_enu_joint: type fixed, parent base_link, child Passive/left_camera_enu_link, origin xyz=0.19 0.075 0.201 rpy=0 0 0
- added joint right_camera_enu_joint: type fixed, parent base_link, child Passive/right_camera_enu_link, origin xyz=0.19 -0.075 0.201 rpy=0 0 0

File: urdf/laboratory/sm2.urdf (robot description, URDF)
Before this commit: robot sm2_mount, 3 links, 2 joints
Links:
- added link SM2/left_camera_enu_link
- added link SM2/right_camera_enu_link
Joints:
- added joint SM2/left_camera_enu_joint: type fixed, parent SM2/base_link, child SM2/left_camera_enu_link, origin xyz=0 0.1 0.0 rpy=0 0 0
- added joint SM2/right_camera_enu_joint: type fixed, parent SM2/base_link, child SM2/right_camera_enu_link, origin xyz=0.0 -0.1 0.0 rpy=0 0 0

Commit message: feat: add ping360 and stim300 link

File: urdf/bluerov2/simple_bluerov2_heavy.urdf (robot description, URDF)
Before this commit: robot bluerov2_heavy, 5 links, 4 joints
Links:
- added link ping360_link
- added link stim3600_link
Joints:
- added joint ping360_joint: type fixed, parent base_link, child ping360_link, origin xyz=0.0 0.0 0.07 rpy=0 0 0
- added joint stim3600_joint: type fixed, parent base_link, child stim3600_link, origin xyz=0.216 0.0 -0.2446 rpy=0 0 0
- joint left_camera_enu_joint: origin xyz=0.19 0.075 0.201 rpy=0 0 0 -> xyz=0.216 0.108 -0.2446 rpy=0 0 0
- joint left_camera_joint: origin xyz=0.19 0.075 0.201 rpy=-1.5707 0 -1.5707 -> xyz=0.216 -0.108 -0.2446 rpy=-1.5707 0 -1.5707
- joint right_camera_enu_joint: origin xyz=0.19 -0.075 0.201 rpy=0 0 0 -> xyz=0.216 -0.108 -0.2446 rpy=0 0 0
- joint right_camera_joint: origin xyz=0.19 -0.075 0.201 rpy=-1.5707 0 -1.5707 -> xyz=0.216 -0.108 -0.2446 rpy=-1.5707 0 -1.5707

Commit message: feat: add new links to blurov2 URDF

File: urdf/bluerov2/simple_bluerov2_heavy.urdf (robot description, URDF)
Before this commit: robot bluerov2_heavy, 7 links, 6 joints
Links:
- added link bluerov2_fpv_link
Joints:
- added joint fpv_joint: type fixed, parent base_link, child bluerov2_fpv_link, origin xyz=0.1 0 0 rpy=-1.5707 0 -1.5707

Commit message: fix: left camera position

File: urdf/bluerov2/simple_bluerov2_heavy.urdf (robot description, URDF)
Before this commit: robot bluerov2_heavy, 8 links, 7 joints
Joints:
- joint fpv_joint: origin xyz=0.1 0 0 rpy=-1.5707 0 -1.5707 -> xyz=0.1 0 0 rpy=-1.5668 0.003 -1.666
- joint left_camera_enu_joint: origin xyz=0.216 0.108 -0.2446 rpy=0 0 0 -> xyz=0.218 0.10728 -0.284 rpy=0 0 0
- joint left_camera_joint: origin xyz=0.216 -0.108 -0.2446 rpy=-1.5707 0 -1.5707 -> xyz=0.218 0.10728 -0.284 rpy=-1.5707 0 -1.5707
- joint right_camera_enu_joint: origin xyz=0.216 -0.108 -0.2446 rpy=0 0 0 -> xyz=0.195 -0.10728 -0.284 rpy=0 0 0
- joint right_camera_joint: origin xyz=0.216 -0.108 -0.2446 rpy=-1.5707 0 -1.5707 -> xyz=0.195 -0.10728 -0.284 rpy=-1.5707 0 -1.5707

Commit message: docs: update rviz2 config file to bluerov

File: urdf/bluerov2/simple_bluerov2_heavy.urdf (robot description, URDF)
Before this commit: robot bluerov2_heavy, 8 links, 7 joints
Links:
- removed link ping360_link
- added link sonar_frame
Joints:
- joint ping360_joint: child ping360_link -> sonar_frame; origin xyz=0.0 0.0 0.07 rpy=0 0 0 -> xyz=0.0 0.0 0.07 rpy=3.14 0 0

Commit message: refactor sonar frame name

File: urdf/bluerov2/simple_bluerov2_heavy.urdf (robot description, URDF)
Before this commit: robot bluerov2_heavy, 8 links, 7 joints
Links:
- removed link sonar_frame
- added link sonar_link
Joints:
- joint ping360_joint: child sonar_frame -> sonar_link

Commit message: fix dvl joint description

File: urdf/bluerov2/simple_bluerov2_heavy.urdf (robot description, URDF)
Before this commit: robot bluerov2_heavy, 8 links, 7 joints
Links:
- added link dvl_link
Joints:
- removed joint ping360_joint
- added joint dvl_joint: type fixed, parent base_link, child dvl_link, origin xyz=-0.075 0.0 -0.3213 rpy=3.14 0 0
- added joint sonar3d_joint: type fixed, parent base_link, child sonar_link, origin xyz=0.13375 0.0 0.1133 rpy=3.14 0 0
